File: noname.sch (KiCad schematic (older format))
At the start: 4 parts

Commit message: Board Updates
Parts:
- removed U? (x4): WS2812B, ~, symbol WS2812B
- added R1, R2, R3, R4: R, symbol R
- added U1, U2, U3, U4: WS2812B, symbol WS2812B
Connections:
- net labels added: VDD, VSS
- wire segments 37 -> 40
Changed lines of the file:
@@
 encoding utf-8
 Sheet 1 1
-Title ""
-Date "26 jun 2014"
+Title "noname.sch"
+Date "26 aug 2014"
 Rev ""
 Comp ""
@@
 $EndDescr
 $Comp
-L WS2812B U?
-U 1 1 53AB97FA
-P 6350 2450
-F 0 "U?" H 5850 2750 60  0000 C CNN
-F 1 "WS2812B" H 5850 2750 60  0000 C CNN
-F 2 "~" H 5850 2750 60  0000 C CNN
-F 3 "~" H 5850 2750 60  0000 C CNN
-	1    6350 2450
-	1    0    0    -1
-$EndComp
-$Comp
-L WS2812B U?
-U 1 1 53AB9809
-P 6350 2900
-F 0 "U?" H 5850 3200 60  0000 C CNN
-F 1 "WS2812B" H 5850 3200 60  0000 C CNN
-F 2 "~" H 5850 3200 60  0000 C CNN
-F 3 "~" H 5850 3200 60  0000 C CNN
-	1    6350 2900
-	1    0    0    -1
-$EndComp
-$Comp
-L WS2812B U?
-U 1 1 53AB9818
-P 6800 2450
-F 0 "U?" H 6300 2750 60  0000 C CNN
-F 1 "WS2812B" H 6300 2750 60  0000 C CNN
-F 2 "~" H 6300 2750 60  0000 C CNN
-F 3 "~" H 6300 2750 60  0000 C CNN
-	1    6800 2450
-	1    0    0    -1
-$EndComp
-$Comp
-L WS2812B U?
-U 1 1 53AB9827
-P 6800 2900
-F 0 "U?" H 6300 3200 60  0000 C CNN
-F 1 "WS2812B" H 6300 3200 60  0000 C CNN
-F 2 "~" H 6300 3200 60  0000 C CNN
-F 3 "~" H 6300 3200 60  0000 C CNN
-	1    6800 2900
-	1    0    0    -1
-$EndComp
-Wire Wire Line
-	5750 2100 5700 2100
-Wire Wire Line
-	5700 2000 5700 2550
-Wire Wire Line
-	6150 1950 6150 2550
-Wire Wire Line
-	6150 2100 6200 2100
-Wire Wire Line
-	5700 2550 5750 2550
-Connection ~ 5700 2100
-Wire Wire Line
-	6150 2550 6200 2550
-Wire Wire Line
-	5950 2650 6000 2650
-Wire Wire Line
-	6000 2200 6000 2750
-Wire Wire Line
-	6400 2650 6450 2650
-Wire Wire Line
-	6450 2750 6450 2200
-Wire Wire Line
-	6450 2200 6400 2200
-Wire Wire Line
-	5950 2200 6000 2200
-Wire Wire Line
-	5650 2750 6500 2750
-Connection ~ 6000 2650
-Connection ~ 6450 2650
-Connection ~ 6150 2100
-Wire Wire Line
-	5750 2200 5650 2200
-Wire Wire Line
-	6200 2650 6100 2650
-Wire Wire Line
-	6100 2650 6100 2450
-Wire Wire Line
-	6200 2200 6050 2200
-Wire Wire Line
-	6050 2200 6050 2350
-Wire Wire Line
-	5650 2650 5750 2650
-Wire Wire Line
-	5650 2450 5650 2650
-Wire Wire Line
-	5950 2550 6050 2550
-Wire Wire Line
-	6050 2550 6050 2400
-Wire Wire Line
-	6050 2400 6500 2400
-Wire Wire Line
-	5950 2100 6100 2100
-Wire Wire Line
-	6100 2100 6100 2350
-Wire Wire Line
-	6100 2350 6500 2350
-Wire Wire Line
-	6400 2100 6500 2100
-Wire Wire Line
-	6500 2100 6500 2300
-Wire Wire Line
-	6400 2550 6500 2550
-Wire Wire Line
-	6500 2550 6500 2450
-Connection ~ 6000 2750
-Connection ~ 6450 2750
-Connection ~ 6150 2000
-Connection ~ 5700 2000
-Wire Wire Line
-	5650 2200 5650 2300
-Connection ~ 5950 2450
-Wire Wire Line
-	6100 2450 5950 2450
-Wire Wire Line
-	5950 2450 5950 2400
-Wire Wire Line
-	5950 2400 5650 2400
-Wire Wire Line
-	6050 2350 5650 2350
-Wire Wire Line
-	5700 2000 6150 2000
-Wire Wire Line
-	5650 1950 6500 1950
-Connection ~ 6150 1950
+L WS2812B U1
+U 1 1 53FC0499
+P 4850 3550
+F 0 "U1" H 4350 3850 60  0000 C CNN
+F 1 "WS2812B" H 4350 3850 60  0000 C CNN
+F 2 "" H 4350 3850 60  0000 C CNN
+F 3 "~" H 4350 3850 60  0000 C CNN
+	1    4850 3550
+	1    0    0    -1
+$EndComp
+$Comp
+L WS2812B U3
+U 1 1 53FC04A8
+P 5250 3550
+F 0 "U3" H 4750 3850 60  0000 C CNN
+F 1 "WS2812B" H 4750 3850 60  0000 C CNN
+F 2 "" H 4750 3850 60  0000 C CNN
+F 3 "~" H 4750 3850 60  0000 C CNN
+	1    5250 3550
+	1    0    0    -1
+$EndComp
+$Comp
+L WS2812B U2
+U 1 1 53FC04B7
+P 4850 3950
+F 0 "U2" H 4350 4250 60  0000 C CNN
+F 1 "WS2812B" H 4350 4250 60  0000 C CNN
+F 2 "" H 4350 4250 60  0000 C CNN
+F 3 "~" H 4350 4250 60  0000 C CNN
+	1    4850 3950
+	1    0    0    -1
+$EndComp
+$Comp
+L WS2812B U4
+U 1 1 53FC04C6
+P 5250 3950
+F 0 "U4" H 4750 4250 60  0000 C CNN
+F 1 "WS2812B" H 4750 4250 60  0000 C CNN
+F 2 "" H 4750 4250 60  0000 C CNN
+F 3 "~" H 4750 4250 60  0000 C CNN
+	1    5250 3950
+	1    0    0    -1
+$EndComp
+Wire Wire Line
+	4850 3200 5050 3200
+Wire Wire Line
+	4650 3200 4600 3200
+Wire Wire Line
+	4600 3200 4600 3100
+Wire Wire Line
+	4250 3200 4200 3200
+Wire Wire Line
+	4200 3200 4200 3100
+Wire Wire Line
+	4450 3200 4550 3200
+Wire Wire Line
+	4550 3200 4550 3250
+Wire Wire Line
+	4550 3250 5050 3250
+Wire Wire Line
+	4450 3300 4400 3300
+Wire Wire Line
+	4400 3300 4400 3400
+Wire Wire Line
+	4650 3300 4500 3300
+Wire Wire Line
+	4500 3300 4500 3250
+Wire Wire Line
+	4500 3250 4150 3250
+Wire Wire Line
+	4250 3300 4150 3300
+Wire Wire Line
+	4250 3700 4150 3700
+Wire Wire Line
+	4850 3600 5050 3600
+Wire Wire Line
+	4450 3600 4550 3600
+Wire Wire Line
+	4550 3600 4550 3650
+Wire Wire Line
+	4550 3650 5050 3650
+Wire Wire Line
+	4650 3600 4600 3600
+Wire Wire Line
+	4600 3600 4600 3500
+Wire Wire Line
+	4250 3600 4200 3600
+Wire Wire Line
+	4200 3600 4200 3500
+Wire Wire Line
+	4850 3300 4900 3300
+Wire Wire Line
+	4900 3300 4900 3400
+Wire Wire Line
+	4400 3400 5100 3400
+Wire Wire Line
+	4650 3700 4500 3700
+Wire Wire Line
+	4500 3700 4500 3650
+Wire Wire Line
+	4500 3650 4150 3650
+Wire Wire Line
+	4450 3700 4450 3800
+Wire Wire Line
+	4450 3800 5100 3800
+Wire Wire Line
+	4900 3800 4900 3700
+Wire Wire Line
+	4900 3700 4850 3700
+$Comp
+L R R3
+U 1 1 53FC06F7
+P 4600 2850
+F 0 "R3" V 4680 2850 40  0000 C CNN
+F 1 "R" V 4607 2851 40  0000 C CNN
+F 2 "" V 4530 2850 30  0000 C CNN
+F 3 "~" H 4600 2850 30  0000 C CNN
+	1    4600 2850
+	1    0    0    -1
+$EndComp
+$Comp
+L R R1
+U 1 1 53FC0710
+P 4200 2850
+F 0 "R1" V 4280 2850 40  0000 C CNN
+F 1 "R" V 4207 2851 40  0000 C CNN
+F 2 "" V 4130 2850 30  0000 C CNN
+F 3 "~" H 4200 2850 30  0000 C CNN
+	1    4200 2850
+	1    0    0    -1
+$EndComp
+$Comp
+L R R2
+U 1 1 53FC071F
+P 4350 3250
+F 0 "R2" V 4430 3250 40  0000 C CNN
+F 1 "R" V 4357 3251 40  0000 C CNN
+F 2 "" V 4280 3250 30  0000 C CNN
+F 3 "~" H 4350 3250 30  0000 C CNN
+	1    4350 3250
+	1    0    0    -1
+$EndComp
+$Comp
+L R R4
+U 1 1 53FC072E
+P 4750 3250
+F 0 "R4" V 4830 3250 40  0000 C CNN
+F 1 "R" V 4757 3251 40  0000 C CNN
+F 2 "" V 4680 3250 30  0000 C CNN
+F 3 "~" H 4750 3250 30  0000 C CNN
+	1    4750 3250
+	1    0    0    -1
+$EndComp
+Wire Wire Line
+	4200 3500 4350 3500
+Wire Wire Line
+	4600 3500 4750 3500
+Wire Wire Line
+	4750 2600 4750 3000
+Wire Wire Line
+	4200 2600 4750 2600
+Wire Wire Line
+	4350 2600 4350 3000
+Connection ~ 4600 2600
+Connection ~ 4350 2600
+$Comp
+L VDD #PWR01
+U 1 1 53FC07F5
+P 4450 2600
+F 0 "#PWR01" H 4450 2700 30  0001 C CNN
+F 1 "VDD" H 4450 2710 30  0000 C CNN
+F 2 "" H 4450 2600 60  0000 C CNN
+F 3 "" H 4450 2600 60  0000 C CNN
+	1    4450 2600
+	1    0    0    -1
+$EndComp
+Connection ~ 4900 3400
+Wire Wire Line
+	5100 3800 5100 3400
+Connection ~ 4900 3800
+$Comp
+L VSS #PWR02
+U 1 1 53FC085A
+P 4550 3850
+F 0 "#PWR02" H 4550 3850 30  0001 C CNN
+F 1 "VSS" H 4550 3780 30  0000 C CNN
+F 2 "" H 4550 3850 60  0000 C CNN
+F 3 "" H 4550 3850 60  0000 C CNN
+	1    4550 3850
+	1    0    0    -1
+$EndComp
+Wire Wire Line
+	4550 3850 4550 3800
+Connection ~ 4550 3800
 $EndSCHEMATC
