File: printed.sch (KiCad schematic (older format))
At the start: 4 parts, among them U1 WS2812B, U2 WS2812B, U3 WS2812B, U4 WS2812B

Commit message: Netlist
Correctly Generated the letlist
Parts:
- added P1, P2: CONN_4, symbol CONN_4
- renumbered U1 to LED1, U2 to LED2, U3 to LED3, U4 to LED4
Connections:
- net at LED1.2 (DOUT): now also P1.4 (P4)
- net at LED1.4 (DIN): now also P2.4 (P4)
- net at LED3.2 (DOUT): now also P1.3 (P3)
- net at LED3.4 (DIN): now also P2.1 (P1)
- net at LED2.2 (DOUT): now also P1.1 (P1)
- net at LED2.4 (DIN): now also P2.2 (P2)
- net at LED4.2 (DOUT): now also P1.2 (P2)
- net at LED4.4 (DIN): now also P2.3 (P3)
- no-connect marks 8 -> 0
Changed lines of the file:
@@
 LIBS:contrib
 LIBS:valves
-LIBS:noname-cache
+LIBS:printed-cache
 EELAYER 27 0
 EELAYER END
@@
 Sheet 1 1
 Title "noname.sch"
-Date "29 aug 2014"
+Date "9 sep 2014"
 Rev ""
 Comp ""
@@
 $EndDescr
 $Comp
-L WS2812B U1
+L WS2812B LED1
 U 1 1 53FFEF12
 P 4700 3300
-F 0 "U1" H 4200 3600 60  0000 C CNN
+F 0 "LED1" H 4200 3600 60  0000 C CNN
 F 1 "WS2812B" H 4200 3600 60  0000 C CNN
 F 2 "~" H 4200 3600 60  0000 C CNN
@@
 $EndComp
 $Comp
-L WS2812B U3
+L WS2812B LED3
 U 1 1 53FFEF21
 P 5250 3300
-F 0 "U3" H 4750 3600 60  0000 C CNN
+F 0 "LED3" H 4750 3600 60  0000 C CNN
 F 1 "WS2812B" H 4750 3600 60  0000 C CNN
 F 2 "~" H 4750 3600 60  0000 C CNN
@@
 $EndComp
 $Comp
-L WS2812B U2
+L WS2812B LED2
 U 1 1 53FFEF30
 P 4700 3700
-F 0 "U2" H 4200 4000 60  0000 C CNN
+F 0 "LED2" H 4200 4000 60  0000 C CNN
 F 1 "WS2812B" H 4200 4000 60  0000 C CNN
 F 2 "~" H 4200 4000 60  0000 C CNN
@@
 $EndComp
 $Comp
-L WS2812B U4
+L WS2812B LED4
 U 1 1 53FFEF3F
 P 5250 3700
-F 0 "U4" H 4750 4000 60  0000 C CNN
+F 0 "LED4" H 4750 4000 60  0000 C CNN
 F 1 "WS2812B" H 4750 4000 60  0000 C CNN
 F 2 "~" H 4750 4000 60  0000 C CNN
@@
 	1    0    0    -1
 $EndComp
-NoConn ~ 4950 3250
-NoConn ~ 4950 3150
-NoConn ~ 4950 3350
-NoConn ~ 4950 3450
-NoConn ~ 3950 3350
-NoConn ~ 3950 3250
-NoConn ~ 3950 3150
-NoConn ~ 3950 3050
 $Comp
 L GND #PWR01
@@
 Connection ~ 4600 2950
 Wire Wire Line
-	4100 3050 3950 3050
-Wire Wire Line
-	3950 3150 4450 3150
+	3850 3050 4100 3050
+Wire Wire Line
+	3850 3150 4450 3150
 Wire Wire Line
 	4100 3450 4000 3450
@@
 	4500 3450 4500 3250
 Wire Wire Line
-	4500 3250 3950 3250
+	4500 3250 3850 3250
 Wire Wire Line
 	4000 3450 4000 3350
 Wire Wire Line
-	4000 3350 3950 3350
+	4000 3350 3850 3350
 Wire Wire Line
 	4400 3050 4400 3700
@@
 Connection ~ 4900 3450
 Wire Wire Line
-	4850 3350 4950 3350
+	4850 3350 5050 3350
 Wire Wire Line
 	4850 2950 4950 2950
@@
 	4050 2950 4100 2950
 Connection ~ 4100 2950
+$Comp
+L CONN_4 P2
+U 1 1 540E8307
+P 5400 3300
+F 0 "P2" V 5350 3300 50  0000 C CNN
+F 1 "CONN_4" V 5450 3300 50  0000 C CNN
+F 2 "" H 5400 3300 60  0000 C CNN
+F 3 "" H 5400 3300 60  0000 C CNN
+	1    5400 3300
+	1    0    0    -1
+$EndComp
+$Comp
+L CONN_4 P1
+U 1 1 540E8316
+P 3500 3200
+F 0 "P1" V 3450 3200 50  0000 C CNN
+F 1 "CONN_4" V 3550 3200 50  0000 C CNN
+F 2 "" H 3500 3200 60  0000 C CNN
+F 3 "" H 3500 3200 60  0000 C CNN
+	1    3500 3200
+	-1   0    0    1
+$EndComp
+Wire Wire Line
+	4950 3150 5050 3150
+Wire Wire Line
+	4950 3250 5050 3250
+Wire Wire Line
+	4950 3450 5050 3450
+Connection ~ 3850 3050
+Connection ~ 3850 3150
+Connection ~ 3850 3250
+Connection ~ 3850 3350
+Connection ~ 5050 3450
+Connection ~ 5050 3350
+Connection ~ 5050 3250
+Connection ~ 5050 3150
 $EndSCHEMATC

Commit message: Headers Added
Parts:
- added P3, P4: CONN_1, symbol CONN_1
Connections:
- net at LED1.1 (VDD), LED2.1 (VDD), LED3.1 (VDD)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: now also P3.1
- net at LED1.3 (VSS), LED2.3 (VSS), LED3.3 (VSS)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: now also P4.1
Changed lines of the file:
@@
 Connection ~ 5050 3250
 Connection ~ 5050 3150
+$Comp
+L CONN_1 P4
+U 1 1 540F1170
+P 4400 3850
+F 0 "P4" H 4480 3850 40  0000 L CNN
+F 1 "CONN_1" H 4400 3905 30  0001 C CNN
+F 2 "" H 4400 3850 60  0000 C CNN
+F 3 "" H 4400 3850 60  0000 C CNN
+	1    4400 3850
+	0    1    1    0
+$EndComp
+$Comp
+L CONN_1 P3
+U 1 1 540F118E
+P 4050 2700
+F 0 "P3" H 4130 2700 40  0000 L CNN
+F 1 "CONN_1" H 4050 2755 30  0001 C CNN
+F 2 "" H 4050 2700 60  0000 C CNN
+F 3 "" H 4050 2700 60  0000 C CNN
+	1    4050 2700
+	0    -1   -1   0
+$EndComp
+Connection ~ 4050 2850
 $EndSCHEMATC

Commit message: Final Schematic,
Nearly to creating the gerber file
Connections:
- net at LED1.4 (DIN): now also P2.2 (P2); no longer P2.4 (P4)
- net at LED2.4 (DIN): now also P2.3 (P3); no longer P2.2 (P2)
- net at LED4.4 (DIN): now also P2.4 (P4); no longer P2.3 (P3)
Changed lines of the file:
@@
 	1    0    0    -1
+$EndComp
+$Comp
+L +5V #PWR02
+U 1 1 540008F4
+P 4050 2850
+F 0 "#PWR02" H 4050 2940 20  0001 C CNN
+F 1 "+5V" H 4050 2940 30  0000 C CNN
+F 2 "" H 4050 2850 60  0000 C CNN
+F 3 "" H 4050 2850 60  0000 C CNN
+	1    4050 2850
+	1    0    0    -1
+$EndComp
+$Comp
+L CONN_4 P2
+U 1 1 540E8307
+P 5400 3300
+F 0 "P2" V 5350 3300 50  0000 C CNN
+F 1 "CONN_4" V 5450 3300 50  0000 C CNN
+F 2 "" H 5400 3300 60  0000 C CNN
+F 3 "" H 5400 3300 60  0000 C CNN
+	1    5400 3300
+	1    0    0    -1
+$EndComp
+$Comp
+L CONN_4 P1
+U 1 1 540E8316
+P 3500 3200
+F 0 "P1" V 3450 3200 50  0000 C CNN
+F 1 "CONN_4" V 3550 3200 50  0000 C CNN
+F 2 "" H 3500 3200 60  0000 C CNN
+F 3 "" H 3500 3200 60  0000 C CNN
+	1    3500 3200
+	-1   0    0    1
+$EndComp
+$Comp
+L CONN_1 P4
+U 1 1 540F1170
+P 4400 3850
+F 0 "P4" H 4480 3850 40  0000 L CNN
+F 1 "CONN_1" H 4400 3905 30  0001 C CNN
+F 2 "" H 4400 3850 60  0000 C CNN
+F 3 "" H 4400 3850 60  0000 C CNN
+	1    4400 3850
+	0    1    1    0
+$EndComp
+$Comp
+L CONN_1 P3
+U 1 1 540F118E
+P 4050 2700
+F 0 "P3" H 4130 2700 40  0000 L CNN
+F 1 "CONN_1" H 4050 2755 30  0001 C CNN
+F 2 "" H 4050 2700 60  0000 C CNN
+F 3 "" H 4050 2700 60  0000 C CNN
+	1    4050 2700
+	0    -1   -1   0
 $EndComp
 Wire Wire Line
@@
 Connection ~ 4900 3450
 Wire Wire Line
-	4850 3350 5050 3350
-Wire Wire Line
 	4850 2950 4950 2950
 Wire Wire Line
 	4950 2950 4950 3150
 Wire Wire Line
-	4300 3350 4450 3350
-Wire Wire Line
-	4450 3350 4450 3200
-Wire Wire Line
-	4450 3200 4950 3200
+	4300 3350 4550 3350
 Wire Wire Line
 	4950 3200 4950 3250
 Wire Wire Line
 	4300 2950 4550 2950
-Wire Wire Line
-	4550 2950 4550 3500
-Wire Wire Line
-	4550 3500 4950 3500
-Wire Wire Line
-	4950 3500 4950 3450
 Connection ~ 4100 3350
 Connection ~ 4100 3450
@@
 	4300 3050 4400 3050
 Connection ~ 4300 3050
-$Comp
-L +5V #PWR02
-U 1 1 540008F4
-P 4050 2850
-F 0 "#PWR02" H 4050 2940 20  0001 C CNN
-F 1 "+5V" H 4050 2940 30  0000 C CNN
-F 2 "" H 4050 2850 60  0000 C CNN
-F 3 "" H 4050 2850 60  0000 C CNN
-	1    4050 2850
-	1    0    0    -1
-$EndComp
 Wire Wire Line
 	4050 2950 4100 2950
 Connection ~ 4100 2950
-$Comp
-L CONN_4 P2
-U 1 1 540E8307
-P 5400 3300
-F 0 "P2" V 5350 3300 50  0000 C CNN
-F 1 "CONN_4" V 5450 3300 50  0000 C CNN
-F 2 "" H 5400 3300 60  0000 C CNN
-F 3 "" H 5400 3300 60  0000 C CNN
-	1    5400 3300
-	1    0    0    -1
-$EndComp
-$Comp
-L CONN_4 P1
-U 1 1 540E8316
-P 3500 3200
-F 0 "P1" V 3450 3200 50  0000 C CNN
-F 1 "CONN_4" V 3550 3200 50  0000 C CNN
-F 2 "" H 3500 3200 60  0000 C CNN
-F 3 "" H 3500 3200 60  0000 C CNN
-	1    3500 3200
-	-1   0    0    1
-$EndComp
 Wire Wire Line
 	4950 3150 5050 3150
 Wire Wire Line
 	4950 3250 5050 3250
-Wire Wire Line
-	4950 3450 5050 3450
 Connection ~ 3850 3050
 Connection ~ 3850 3150
@@
 Connection ~ 5050 3250
 Connection ~ 5050 3150
-$Comp
-L CONN_1 P4
-U 1 1 540F1170
-P 4400 3850
-F 0 "P4" H 4480 3850 40  0000 L CNN
-F 1 "CONN_1" H 4400 3905 30  0001 C CNN
-F 2 "" H 4400 3850 60  0000 C CNN
-F 3 "" H 4400 3850 60  0000 C CNN
-	1    4400 3850
-	0    1    1    0
-$EndComp
-$Comp
-L CONN_1 P3
-U 1 1 540F118E
-P 4050 2700
-F 0 "P3" H 4130 2700 40  0000 L CNN
-F 1 "CONN_1" H 4050 2755 30  0001 C CNN
-F 2 "" H 4050 2700 60  0000 C CNN
-F 3 "" H 4050 2700 60  0000 C CNN
-	1    4050 2700
-	0    -1   -1   0
-$EndComp
 Connection ~ 4050 2850
+Wire Wire Line
+	4550 2950 4550 3200
+Wire Wire Line
+	4550 3200 4950 3200
+Wire Wire Line
+	4550 3350 4550 3250
+Wire Wire Line
+	4550 3250 4850 3250
+Wire Wire Line
+	4850 3350 4950 3350
+Wire Wire Line
+	4950 3350 4950 3450
+Wire Wire Line
+	4950 3450 5050 3450
+Wire Wire Line
+	4850 3250 4850 3300
+Wire Wire Line
+	4850 3300 5050 3300
+Wire Wire Line
+	5050 3300 5050 3350
 $EndSCHEMATC
